File: pcbs/ATtiny_board/ATtiny_board.kicad_pcb (KiCad board)
At the start: 2 copper layers, 2 parts, among them U1 ATtiny85V-10PU

Commit message: Continued PCB
Parts:
- added C1: 1F 5.5V, ivo_lib:1FSuperCap, F.Cu at (149.9, 71.1)
- added C2: 440μF, Capacitor_THT:C_Disc_D4.3mm_W1.9mm_P5.00mm, F.Cu at (134.6, 93.9)
- added C3: 0.1μF, Capacitor_THT:C_Disc_D4.3mm_W1.9mm_P5.00mm, F.Cu at (124.5, 100.5)
- added D1: LED, Diode_THT:D_A-405_P2.54mm_Vertical_AnodeUp, F.Cu at (119.4, 83.8)
- added J1: To reedswitch, Connector_PinHeader_2.54mm:PinHeader_1x02_P2.54mm_Vertical, F.Cu at (152.4, 91.4)
- added R1: 330Ω, Resistor_THT:R_Axial_DIN0207_L6.3mm_D2.5mm_P10.16mm_Horizontal, F.Cu at (123.4, 84.0)
- added R2: 1.8kΩ, Resistor_THT:R_Axial_DIN0207_L6.3mm_D2.5mm_P10.16mm_Horizontal, F.Cu at (147.3, 88.9)
- added SC1: KXOB25-05X3F, ivo_lib:KXOB25-05X3F, F.Cu at (124.5, 50.8)
- added SW2: Display Switch, Button_Switch_THT:SW_PUSH_6mm, F.Cu at (134.9, 107.4)
- moved U1 16.9 mm to (132.1, 96.6), turned to 180 degrees
- moved U2 14.7 mm to (124.5, 68.6)
Connections:
- U2 pad 1: Net-(U2-CFG2) -> unconnected-(U2-GND-Pad1)
- U2 pad 6: Net-(U2-SELMPP[1]) -> Net-(U2-CFG2)
- U2 pad 7: Net-(U2-SELMPP[1]) -> Net-(U2-CFG2)
Routing:
- net Net-(U1-GND): track 0.00 -> 44.6 mm
- net Net-(U2-BUCK): track 0.00 -> 40.5 mm
- net Net-(U1-VCC): track 0.00 -> 25.8 mm
- net Net-(J1-Pin_1): track 0.00 -> 21.4 mm
- net Net-(U2-BAT): track 0.00 -> 18.1 mm
- net Net-(U1-XTAL2/PB4): track 0.00 -> 15.0 mm
- net Net-(U2-CFG2): track 0.00 -> 9.52 mm
- net Net-(D1-A): track 0.00 -> 6.15 mm
- net Net-(J1-Pin_2): track 0.00 -> 5.08 mm
- net Net-(D1-K): track 0.00 -> 4.09 mm
- net Net-(U2-ENLV): track 0.00 -> 2.40 mm
- net Net-(SC1-+): track 0.00 -> 2.06 mm
- net Net-(SC1--): track 0.00 -> 1.92 mm
- added copper zone on B.Cu, net Net-(U1-GND)
Other:
- board text added: "+ve"
- board text added: "-ve"
