File: pcbs/ATtiny_board/ATtiny_board.kicad_sch (KiCad schematic)
At the start: 1 part, among them U1 ATtiny85V-10P

Commit message: Designing PCB
Parts:
- added C1: 1F 5.5V, symbol Device:C_Polarized
- added C2: 440μF, symbol Device:C_Small
- added D1: LED, symbol Device:LED
- added R1: 330Ω, symbol Device:R
- added R2: 1.8kΩ, symbol Device:R
- added SC1: KXOB25-05X3F, symbol Device:Solar_Cells
- added SW1: (no value), symbol Switch:SW_Reed
- added SW2: Display Switch, symbol Switch:SW_Push
- added U2: (no value), energy_harvest:AEM10941_board, symbol new_ivo_lib:AEM10941_board
- U1: value ATtiny85V-10P -> ATtiny85V-10PU
Connections:
- net at U1.2 (XTAL1/PB3): now also C2.1, SW1.2
- net at U1.3 (XTAL2/PB4): now also SW2.1
- net at U1.4 (GND): now also C1.2, C2.2, R1.2, R2.2, SW2.2, U2.16 (GND), U2.17 (BAL)
- net at U1.5 (AREF/PB0): now also D1.2 (A)
- net at U1.6 (PB1): now also U2.23 (STATUS[1])
- net at U1.8 (VCC): now also U2.15 (HVOUT)
- new net: R2.1, SW1.1
- new net: D1.1 (K), R1.1
- new net: U2.1 (GND), U2.3 (CFG2)
- new net: U2.10 (FB_PRIM_U), U2.11 (GND), U2.9 (FB_PRIM_D)
- new net: U2.13 (ENHV), U2.2 (BUCK), U2.26 (SET_OVCH), U2.27 (SET_CHRDY), U2.28 (SET_OVDIS), U2.4 (CFG1), U2.5 (CFG0), U2.8 (SELMPP[0])
- new net: C1.1, U2.18 (BAT)
- new net: U2.19 (PRIM), U2.20 (ENLV), U2.21 (GND)
- new net: SC1.1 (+), U2.29 (SRC)
- new net: SC1.2 (-), U2.30 (GND)
- new net: U2.6 (GND), U2.7 (SELMPP[1])
Other:
- note added: "AEM10941"
- moved on the sheet: U1

Commit message: Continued PCB
Parts:
- removed SW1: (no value), symbol Switch:SW_Reed
- added C3: 0.1μF, Capacitor_THT:C_Disc_D4.3mm_W1.9mm_P5.00mm, symbol Device:C_Small
- added J1: To reedswitch, Connector_PinHeader_2.54mm:PinHeader_1x02_P2.54mm_Vertical, symbol Connector:Conn_01x02_Socket
- C1: footprint (none) -> ivo_lib:1FSuperCap
- C2: footprint (none) -> Capacitor_THT:C_Disc_D4.3mm_W1.9mm_P5.00mm
- D1: footprint (none) -> Diode_THT:D_A-405_P2.54mm_Vertical_AnodeUp
- R1, R2: footprint (none) -> Resistor_THT:R_Axial_DIN0207_L6.3mm_D2.5mm_P10.16mm_Horizontal
- SC1: footprint (none) -> ivo_lib:KXOB25-05X3F
- SW2: footprint (none) -> Button_Switch_THT:SW_PUSH_6mm
Connections:
- net at R2.1: now also J1.2 (Pin_2)
- net at C1.2, C2.2, R1.2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: now also C3.2
- net at U2.1 (GND): no longer U2.3 (CFG2)
- net at U1.8 (VCC), U2.15 (HVOUT): now also C3.1
- net at U2.6 (GND), U2.7 (SELMPP[1]): now also U2.3 (CFG2)
- net at C2.1, U1.2 (XTAL1/PB3): now also J1.1 (Pin_1)
Other:
- added sheet Reed Switch (untitled.kicad_sch)
